File: NixieDriver.kicad_sch (KiCad schematic)
At the start: 0 parts

Commit message: add git hash
Other:
- title: (none) -> ZM108x, Z57x nixieboard
Changed lines of the file:
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@@
 (kicad_sch (version 20230121) (generator eeschema)
   (paper "A4")
+  (title_block
+    (title "ZM108x, Z57x nixieboard")
+    (date "2025-09-04")
+    (rev "3/${GITHASH}")
+    (comment 1 "Atuthor: Martin Sabol")
+  )
   (junction (at 85.09 100.33) (diameter 0) (color 0 0 0 0)
   )
