File: neon.kicad_sch (KiCad schematic)
At the start: 4 parts, among them Q1101 PMBTA42

Commit message: add git hash
Other:
- title: (none) -> ZM108x, Z57x nixieboard
Changed lines of the file:
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@@
 (kicad_sch (version 20230121) (generator eeschema)
   (paper "A4")
+  (title_block
+    (title "ZM108x, Z57x nixieboard")
+    (date "2025-09-04")
+    (rev "3/${GITHASH}")
+    (comment 1 "Atuthor: Martin Sabol")
+  )
   (wire (pts (xy 146.05 109.22) (xy 151.13 109.22))
     (stroke (width 0) (type default))

Commit message: schema: bom: PNs update
Parts:
- Q1101: SPN PMBTA42 -> PMBTA42,215
- R1101: SPN RC0603FR-073K3 -> RC0201FR-073K3L
- R1102: SPN SMD1206-120K-1% -> 1206S4F1203T5E
Changed lines of the file:
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@@
       (effects (font (size 1.27 1.27)) (justify left) hide)
     )
-    (property "SPN" "PMBTA42" (at 156.21 109.22 0)
+    (property "SPN" "PMBTA42,215" (at 156.21 109.22 0)
       (effects (font (size 1.27 1.27)) (justify left) hide)
     )
@@
       (effects (font (size 1.27 1.27)) hide)
     )
-    (property "SPN" "RC0603FR-073K3" (at 142.24 109.22 0)
+    (property "SPN" "RC0201FR-073K3L" (at 142.24 109.22 0)
       (effects (font (size 1.27 1.27)) hide)
     )
@@
       (effects (font (size 1.27 1.27)) hide)
     )
-    (property "SPN" "SMD1206-120K-1%" (at 158.75 82.55 0)
+    (property "SPN" "1206S4F1203T5E" (at 158.75 82.55 0)
       (effects (font (size 1.27 1.27)) hide)
     )

Commit message: BoM: optimize parts
Parts:
- R1101: SPN RC0201FR-073K3L -> 0603SAF3301T5E
Changed lines of the file:
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@@
       (effects (font (size 1.27 1.27)) hide)
     )
-    (property "SPN" "RC0201FR-073K3L" (at 142.24 109.22 0)
+    (property "SPN" "0603SAF3301T5E" (at 142.24 109.22 0)
       (effects (font (size 1.27 1.27)) hide)
     )
