File: nixieboard.kicad_sch (KiCad schematic)
At the start: 19 parts, among them J101 USB4110-GF-A, J102 DEBUG_UART, SW101 SW_Push, SW102 SW_Push

Commit message: add git hash
Other:
- title: (none) -> ZM108x, Z57x nixieboard
Changed lines of the file:
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@@
 (kicad_sch (version 20230121) (generator eeschema)
   (paper "A4")
+  (title_block
+    (title "ZM108x, Z57x nixieboard")
+    (date "2025-09-04")
+    (rev "3/${GITHASH}")
+    (comment 1 "Atuthor: Martin Sabol")
+  )
   (junction (at 86.36 118.11) (diameter 0) (color 0 0 0 0)
   )

Commit message: schema: bom: PNs update
Parts:
- C101, C102: SPN CL10B105KO8NNNC -> CL21B105KOFNNNE
- J101: SPN (none) -> USB4110-GF-A
- J102: SPN (none) -> 53261-0471
- R101: SPN RC0603FR-073K3 -> 0805S8F3301T5E
- R102, R103: SPN RC0603FR-073K3 -> 0805S8F5101T5E
- R104, R105: SPN RC0603FR-073K3 -> 0805S8F270JT5E
- SW101, SW102: SPN DTSM-66S-V-B -> DTSM-66R-V-B
Changed lines of the file:
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@@
       (effects (font (size 1.27 1.27)) hide)
     )
-    (property "SPN" "DTSM-66S-V-B" (at 152.4 97.79 0)
+    (property "SPN" "DTSM-66R-V-B" (at 152.4 97.79 0)
       (effects (font (size 1.27 1.27)) hide)
     )
@@
       (effects (font (size 1.27 1.27)) hide)
     )
-    (property "SPN" "DTSM-66S-V-B" (at 152.4 107.95 0)
+    (property "SPN" "DTSM-66R-V-B" (at 152.4 107.95 0)
       (effects (font (size 1.27 1.27)) hide)
     )
@@
       (effects (font (size 1.27 1.27)) hide)
     )
-    (property "SPN" "RC0603FR-073K3" (at 35.56 144.78 0)
+    (property "SPN" "0805S8F3301T5E" (at 35.56 144.78 0)
       (effects (font (size 1.27 1.27)) hide)
     )
@@
       (effects (font (size 1.27 1.27)) hide)
     )
-    (property "SPN" "CL10B105KO8NNNC" (at 26.67 144.78 0)
+    (property "SPN" "CL21B105KOFNNNE" (at 26.67 144.78 0)
       (effects (font (size 1.27 1.27)) hide)
     )
@@
       (effects (font (size 1.27 1.27)) hide)
     )
-    (property "SPN" "CL10B105KO8NNNC" (at 86.36 123.19 0)
+    (property "SPN" "CL21B105KOFNNNE" (at 86.36 123.19 0)
       (effects (font (size 1.27 1.27)) hide)
     )
@@
     )
     (property "Datasheet" "https://www.usb.org/sites/default/files/documents/usb_type-c.zip" (at 46.99 105.41 0)
+      (effects (font (size 1.27 1.27)) hide)
+    )
+    (property "SPN" "USB4110-GF-A" (at 43.18 105.41 0)
       (effects (font (size 1.27 1.27)) hide)
     )
@@
       (effects (font (size 1.27 1.27)) hide)
     )
-    (property "SPN" "RC0603FR-073K3" (at 74.93 147.32 0)
+    (property "SPN" "0805S8F5101T5E" (at 74.93 147.32 0)
       (effects (font (size 1.27 1.27)) hide)
     )
@@
       (effects (font (size 1.27 1.27)) hide)
     )
-    (property "SPN" "RC0603FR-073K3" (at 110.49 107.95 0)
+    (property "SPN" "0805S8F270JT5E" (at 110.49 107.95 0)
       (effects (font (size 1.27 1.27)) hide)
     )
@@
       (effects (font (size 1.27 1.27)) hide)
     )
-    (property "SPN" "RC0603FR-073K3" (at 68.58 147.32 0)
+    (property "SPN" "0805S8F5101T5E" (at 68.58 147.32 0)
       (effects (font (size 1.27 1.27)) hide)
     )
@@
       (effects (font (size 1.27 1.27)) hide)
     )
-    (property "SPN" "RC0603FR-073K3" (at 110.49 102.87 0)
+    (property "SPN" "0805S8F270JT5E" (at 110.49 102.87 0)
       (effects (font (size 1.27 1.27)) hide)
     )
@@
       (effects (font (size 1.27 1.27)) hide)
     )
+    (property "SPN" "53261-0471" (at 204.47 113.03 0)
+      (effects (font (size 1.27 1.27)) hide)
+    )

Commit message: BoM: optimize parts
Parts:
- C101, C102: value 1u -> 1u/16V
Changed lines of the file:
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@@
       (effects (font (size 1.27 1.27)) (justify left))
     )
-    (property "Value" "1u" (at 27.305 147.32 0)
+    (property "Value" "1u/16V" (at 27.305 147.32 0)
       (effects (font (size 1.27 1.27)) (justify left))
     )
@@
       (effects (font (size 1.27 1.27)) (justify left))
     )
-    (property "Value" "1u" (at 86.995 125.73 0)
+    (property "Value" "1u/16V" (at 86.995 125.73 0)
       (effects (font (size 1.27 1.27)) (justify left))
     )
